File: PCB/TTL2ANALOG.kicad_pcb (KiCad board)
At the start: 2 copper layers, 59.7 x 45.1 mm, 23 parts, among them J1 EGA Input, J3 CSync Selection, J4 Power, J5 Video Out, U1 27C010, U2 74LS244

Commit message: Begin drawing PCB
Parts:
- removed F1: 250mA, Fuse:Fuse_1206_3216Metric
- removed JP1: EGA/CGA, Connector_PinHeader_2.54mm:PinHeader_1x02_P2.54mm_Vertical
- removed JP2: Brown Fix, Connector_PinHeader_2.54mm:PinHeader_1x02_P2.54mm_Vertical
- added C1: 22pF, Capacitor_SMD:C_1206_3216Metric_Pad1.33x1.80mm_HandSolder, F.Cu at (59.4, 61.5)
- added C2: 22pF, Capacitor_SMD:C_1206_3216Metric_Pad1.33x1.80mm_HandSolder, F.Cu at (82.5, 40.2)
- added C3: 22pF, Capacitor_SMD:C_1206_3216Metric_Pad1.33x1.80mm_HandSolder, F.Cu at (65.4, 61.5)
- added C6: 100nF, Capacitor_SMD:C_1206_3216Metric_Pad1.33x1.80mm_HandSolder, F.Cu at (82.5, 43.5)
- added C7: 10uF, Capacitor_THT:CP_Radial_D7.5mm_P2.50mm, F.Cu at (59.9, 54.8)
- added C8: 100nF, Capacitor_SMD:C_1206_3216Metric_Pad1.33x1.80mm_HandSolder, F.Cu at (82.5, 46.9)
- added J2: Brown Fix, Connector_PinSocket_2.54mm:PinSocket_1x03_P2.54mm_Vertical, F.Cu at (54.2, 52.6)
- added J6: Analog Out, Connector_Dsub:DSUB-15-HD_Female_Horizontal_P2.29x1.98mm_EdgePinOffset3.03mm_Housed_MountingHolesOffset4.94mm, F.Cu at (55.6, 35.8)
- added J7: Barrel_Jack, Connector_BarrelJack:BarrelJack_Horizontal, F.Cu at (114.9, 97.5)
- added U3: 74LS244, Package_DIP:DIP-20_W7.62mm_Socket, F.Cu at (69.8, 34.8)
- added U4: L78L05_TO92, Package_TO_SOT_THT:TO-92_Inline, F.Cu at (81.5, 35.9)
- C4, C5: footprint Capacitor_THT:C_Disc_D3.0mm_W2.0mm_P2.50mm -> Capacitor_SMD:C_1206_3216Metric_Pad1.33x1.80mm_HandSolder
- D1: value 1N4733A -> 1N4001
- D2: footprint LED_THT:LED_D2.0mm_W4.8mm_H2.5mm_FlatTop -> LED_SMD:LED_0805_2012Metric_Pad1.15x1.40mm_HandSolder
- J1: value EGA Input -> EGA/CGA; footprint Connector_Dsub:DSUB-9_Female_Horizontal_P2.77x2.84mm_EdgePinOffset4.94mm_Housed_MountingHolesOffset7.48mm -> Connector_PinSocket_2.54mm:PinSocket_1x03_P2.54mm_Vertical
- J4: value Power -> Sync Type; footprint TerminalBlock:TerminalBlock_bornier-2_P5.08mm -> Connector_PinSocket_2.54mm:PinSocket_1x03_P2.54mm_Vertical
- J5: value Video Out -> TTL Input; footprint TerminalBlock:TerminalBlock_bornier-6_P5.08mm -> Connector_Dsub:DSUB-9_Female_Horizontal_P2.77x2.84mm_EdgePinOffset4.94mm_Housed_MountingHolesOffset7.48mm
- R10, R2, R3, R4, R5, R7: footprint Resistor_THT:R_Axial_DIN0204_L3.6mm_D1.6mm_P7.62mm_Horizontal -> Resistor_SMD:R_1206_3216Metric_Pad1.30x1.75mm_HandSolder
- R8, R9: value 4.7k -> 10k
- U1: value 27C010 -> GAL16V8; footprint Package_DIP:DIP-32_W15.24mm -> Package_DIP:DIP-20_W7.62mm_Socket
- U2: footprint Package_DIP:DIP-20_W7.62mm -> Package_DIP:DIP-20_W7.62mm_Socket
- moved D1 44.8 mm to (107.6, 94.7), turned to 270 degrees
- moved J5 21.2 mm to (149.2, 98.9), turned to 0 degrees
Connections:
- D1 pad 1: VCC -> Net-(C7-Pad1)
- D1 pad 2: GND -> Net-(D1-Pad2)
- J1 pad 2: /IN_R_I -> /MODE
- J1 pad 3: /IN_R -> (no net)
- J4 pad 1: Net-(F1-Pad2) -> /IN_VS_BUF
- J4 pad 2: GND -> /SYNC_OUT
- J5 pad 1: /ANALOG_R -> GND
- J5 pad 2: /ANALOG_G -> /IN_R_I
- J5 pad 3: /ANALOG_B -> /IN_R
- J5 pad 4: /ANALOG_CSYNC -> /IN_G
- J5 pad 5: GND -> /IN_B
- J5 pad 6: GND -> /IN_G_I
- R8 pad 1: /MODE_IN -> VCC
- R8 pad 2: VCC -> /BRWN_FIX
- R9 pad 1: GND -> VCC
- R9 pad 2: Net-(JP2-Pad2) -> /MODE
- U1 pad 1: VCC -> /IN_G_I_BUF
- U1 pad 10: /IN_B_I -> GND
- U1 pad 11: /IN_B -> /BRWN_FIX
- U1 pad 12: /MODE_IN -> /~DEC_CS
- U1 pad 13: /DEC_B -> /DEC_CS
- U1 pad 14: /DEC_B_I -> /DEC_R_I
- U1 pad 15: /DEC_G -> /DEC_R
- U1 pad 16: GND -> /DEC_G_I
- U1 pad 17: /DEC_G_I -> /DEC_G
- U1 pad 18: /DEC_R -> /DEC_B_I
- U1 pad 19: /DEC_R_I -> /DEC_B
- U1 pad 2: GND -> /IN_R_I_BUF
- U1 pad 20: /DEC_CS -> VCC
- U1 pad 3: GND -> /IN_B_I_BUF
- U1 pad 4: GND -> /IN_R_BUF
- U1 pad 5: /IN_VS -> /IN_HS_BUF
- U1 pad 6: /IN_R_I -> /IN_G_BUF
- U1 pad 7: /IN_R -> /IN_VS_BUF
- U1 pad 8: /IN_G_I -> /IN_B_BUF
- U1 pad 9: /IN_G -> /MODE
Routing:
- net GND: track 185.7 -> 0.00 mm
- net VCC: track 135.6 -> 0.00 mm
- net /DEC_B: track 55.2 -> 0.00 mm
- net /OUT_G_I: track 47.4 -> 0.00 mm
- net /OUT_R: track 40.1 -> 0.00 mm
- net /OUT_R_I: track 36.9 -> 0.00 mm
- net /IN_HS: track 33.0 -> 0.00 mm
- net /OUT_G: track 32.8 -> 0.00 mm, vias 1 -> 0
- net Net-(JP2-Pad2): track 32.4 -> 0.00 mm
- net /DEC_B_I: track 30.1 -> 0.00 mm
- net /MODE_IN: track 28.5 -> 0.00 mm
- net /OUT_B: track 24.7 -> 0.00 mm
- net /DEC_G: track 24.1 -> 0.00 mm
- net /IN_R_I: track 20.5 -> 0.00 mm
- net /OUT_B_I: track 19.9 -> 0.00 mm
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- removed copper zone on B.Cu, net GND
- removed copper zone on F.Cu, net GND
Other:
- board outline removed
- board text removed: "+"
- board text removed: "-"
- board text removed: "5Vdc"
- board text removed: "EGA-2-RGBS"
- board text removed: "R"
- board text removed: "rev 1.1"
