File: PCB/TTL2ANALOG.kicad_sch (KiCad schematic)
At the start: 38 parts, among them J1 EGA/CGA, J2 Options, J3 CSync Inv., J4 Sync Type, J5 TTL Input, J6 Analog Out, J7 Barrel_Jack, U1 GAL20V8, U2 74LS244, U3 74LS244, U4 L7805

Commit message: Redraw version 1.4
Parts:
- removed C7: 10uF, Capacitor_THT:CP_Radial_D6.3mm_P2.50mm, symbol Device:C_Polarized_Small
- removed H1, H2, H3, H4: MountingHole_Pad, MountingHole:MountingHole_3.2mm_M3_DIN965_Pad, symbol Mechanical:MountingHole_Pad
- removed J1: EGA/CGA, Connector_PinHeader_2.54mm:PinHeader_1x03_P2.54mm_Vertical, symbol Connector_Generic:Conn_01x03
- removed U4: L7805, Package_TO_SOT_THT:TO-220-3_Vertical, symbol Regulator_Linear:L7805
- added C7: 10uF, Capacitor_SMD:C_1206_3216Metric_Pad1.33x1.80mm_HandSolder, symbol Device:C_Small
- added U5: AMS1117-5.0, Package_TO_SOT_SMD:SOT-223-3_TabPin2, symbol Regulator_Linear:AMS1117-5.0
- C8: value 100nF -> 10uF
- D2: footprint LED_SMD:LED_0805_2012Metric_Pad1.15x1.40mm_HandSolder -> LED_SMD:LED_1206_3216Metric_Pad1.42x1.75mm_HandSolder
Connections:
- net BRWN_FIX: now also J2.7 (Pin_7), RN2.3 (R2); no longer J2.4 (Pin_4), RN2.5 (R4)
- net GND: now also C7.2, U5.1 (GND)
- net IN_B: now also RN1.5 (R4); no longer RN1.2 (R1)
- net IN_G: now also RN1.3 (R2); no longer RN1.4 (R3)
- net IN_HS: now also RN1.2 (R1); no longer RN1.5 (R4)
- net IN_VS: now also RN1.4 (R3); no longer RN1.3 (R2)
- net MODE: now also J2.5 (Pin_5), RN2.4 (R3); no longer J2.2 (Pin_2), RN2.6 (R5)
- net VCC: now also J2.10 (Pin_10), J2.2 (Pin_2), J2.4 (Pin_4), J2.6 (Pin_6), J2.8 (Pin_8), U5.2 (VO); no longer J2.1 (Pin_1), J2.3 (Pin_3), J2.5 (Pin_5), J2.7 (Pin_7), J2.9 (Pin_9)
- net at D1.1 (K): now also C7.1, U5.3 (VI)
- net at RN2.2 (R1), U1.23 (I23): now also J2.9 (Pin_9); no longer J2.10 (Pin_10)
- new net: J2.1 (Pin_1), RN2.6 (R5), U1.13 (I13)
- new net: J2.3 (Pin_3), RN2.5 (R4), U1.14 (I14)
- no-connect marks 5 -> 4
Other:
- moved on the sheet: J5, RN1, RN2
